File: 001_Analoge_Schaltungen/schaltungsentwurf_no1/_autosave-schaltungsentwurf_no1.kicad_sch (KiCad schematic)
At the start: 15 parts, among them U1 TL082, U2 TL082

Commit message: chore:add untracked files
Parts:
- R2, R3: value {RCOM} -> {RF}
Other:
- note added: ".param RCOM = 1k .param RF = 900 .param CCOM = 1u .param Q = 10 .param H0 = 1"
- note removed: ".param RCOM = 1k .param CCOM = 1u .param Q = 5 .param H0 = 1"
Changed lines of the file:
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@@
 		)
 	)
-	(text ".param RCOM = 1k\n.param CCOM = 1u\n.param Q = 5\n.param H0 = 1\n\n"
+	(text ".param RCOM = 1k\n.param RF = 900\n.param CCOM = 1u\n.param Q = 10\n.param H0 = 1\n\n"
 		(exclude_from_sim no)
 		(at 190.246 86.868 0)
@@
 			)
 		)
-		(property "Value" "{RCOM}"
+		(property "Value" "{RF}"
 			(at 73.66 44.45 90)
 			(effects
@@
 			)
 		)
-		(property "Value" "{RCOM}"
+		(property "Value" "{RF}"
 			(at 114.3 46.99 90)
 			(effects
